File: kicad/pico-radio-5/pico-radio-5.kicad_sch (KiCad schematic)
At the start: 44 parts, among them J1 HF Amplifier, J2 MW/SW antenna, J3 FM antenna, J4 SW antenna, J5 Batterry, Q1 PN2222A, Q2 PN2222A, Q3 PN2222A, SW1 Reset, U1 SI4732-A10-GS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

Commit message: Refactor code structure for improved readability and maintainability
Parts:
- added JP3: TFT SDO - ha kell, Jumper:SolderJumper-2_P1.3mm_Open_RoundedPad1.0x1.5mm, symbol Jumper:SolderJumper_2_Open
- L1: value 47uH -> 220uH
- L2: value 270uH -> 220uH
- R1: value 200k -> 10k
- R2: value 100k -> 15k
Connections:
- net +3.3V: no longer BZ1.1 (+)
- net +Vbus: now also BZ1.1 (+)
- net SDO: now also JP3.2 (B); no longer U2.9 (SDO/MISO)
- new net: JP3.1 (A), U2.9 (SDO/MISO)
Other:
- note added: "A TFT SDO/MISO bekötése opcionális! Akkor kell, ha a TFT-ről pixel adatokat szeretnénk beolvasni"
Changed lines of the file:
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@@
 		(date "2025-08-04")
 	)
+	(text "A TFT SDO/MISO bekötése opcionális!\nAkkor kell, ha a TFT-ről pixel adatokat szeretnénk beolvasni"
+		(exclude_from_sim no)
+		(at 13.97 15.748 0)
+		(effects
+			(font
+				(size 1.27 1.27)
+			)
+			(justify left)
+		)
+	)
 	(junction
 		(at 168.91 111.76)
@@
 	)
 	(bus_entry
+		(at 102.87 49.53)
+		(size 2.54 2.54)
+		(stroke
+			(width 0)
+			(type default)
+		)
+	)
+	(bus_entry
 		(at 88.9 71.12)
 		(size 2.54 2.54)
@@
 	)
 	(bus_entry
-		(at 99.06 71.12)
+		(at 104.14 71.12)
 		(size 2.54 2.54)
 		(stroke
@@
 	)
 	(bus_entry
-		(at 104.14 71.12)
+		(at 139.7 64.77)
 		(size 2.54 2.54)
 		(stroke
@@
 	(bus
 		(pts
-			(xy 128.27 43.18) (xy 128.27 73.66)
+			(xy 142.24 43.18) (xy 142.24 67.31)
+		)
+		(stroke
+			(width 0)
+			(type default)
+		)
+	)
+	(wire
+		(pts
+			(xy 251.46 92.71) (xy 251.46 100.33)
 		)
 		(stroke
@@
 	(wire
 		(pts
+			(xy 99.06 64.77) (xy 99.06 62.23)
+		)
+		(stroke
+			(width 0)
+			(type default)
+		)
+	)
+	(wire
+		(pts
 			(xy 22.86 73.66) (xy 22.86 72.39)
 		)
@@
 	(wire
 		(pts
-			(xy 251.46 97.79) (xy 251.46 100.33)
-		)
-		(stroke
-			(width 0)
-			(type default)
-		)
-	)
-	(wire
-		(pts
 			(xy 262.89 139.7) (xy 266.7 139.7)
 		)
@@
 		)
 	)
+	(bus
+		(pts
+			(xy 142.24 67.31) (xy 142.24 73.66)
+		)
+		(stroke
+			(width 0)
+			(type default)
+		)
+	)
 	(wire
 		(pts
@@
 	(wire
 		(pts
+			(xy 124.46 64.77) (xy 99.06 64.77)
+		)
+		(stroke
+			(width 0)
+			(type default)
+		)
+	)
+	(wire
+		(pts
 			(xy 135.89 173.99) (xy 135.89 181.61)
 		)
@@
 	(bus
 		(pts
-			(xy 99.06 73.66) (xy 101.6 73.66)
+			(xy 99.06 73.66) (xy 104.14 73.66)
 		)
 		(stroke
@@
 	(bus
 		(pts
-			(xy 128.27 73.66) (xy 111.76 73.66)
+			(xy 142.24 73.66) (xy 111.76 73.66)
 		)
 		(stroke
@@
 		)
 	)
-	(bus
-		(pts
-			(xy 101.6 73.66) (xy 104.14 73.66)
-		)
-		(stroke
-			(width 0)
-			(type default)
-		)
-	)
 	(wire
 		(pts
@@
 	(wire
 		(pts
+			(xy 132.08 64.77) (xy 139.7 64.77)
+		)
+		(stroke
+			(width 0)
+			(type default)
+		)
+	)
+	(wire
+		(pts
 			(xy 251.46 119.38) (xy 251.46 123.19)
 		)
@@
 	(wire
 		(pts
-			(xy 99.06 62.23) (xy 99.06 71.12)
-		)
-		(stroke
-			(width 0)
-			(type default)
-		)
-	)
-	(wire
-		(pts
 			(xy 107.95 95.25) (xy 116.84 95.25)
 		)
@@
 	(bus
 		(pts
-			(xy 128.27 43.18) (xy 151.13 43.18)
+			(xy 142.24 43.18) (xy 151.13 43.18)
 		)
 		(stroke
@@
 		)
 	)
-	(label "SDO"
-		(at 99.06 71.12 90)
-		(effects
-			(font
-				(size 1.27 1.27)
-			)
-			(justify left bottom)
-		)
-	)
 	(label "SDI"
 		(at 91.44 71.12 90)
@@
 		)
 	)
+	(label "SDO"
+		(at 135.89 64.77 0)
+		(effects
+			(font
+				(size 1.27 1.27)
+			)
+			(justify left bottom)
+		)
+	)
 	(label "SCK"
 		(at 101.6 71.12 90)
@@
 	)
 	(symbol
-		(lib_id "power:+3.3V")
-		(at 251.46 97.79 0)
-		(unit 1)
-		(exclude_from_sim no)
-		(in_bom yes)
-		(on_board yes)
-		(dnp no)
-		(property "Reference" "#PWR011"
-			(at 251.46 101.6 0)
-			(effects
-				(font
-					(size 1.27 1.27)
-				)
-				(hide yes)
-			)
-		)
-		(property "Value" "+3.3V"
-			(at 255.524 96.012 0)
-			(effects
-				(font
-					(size 1.27 1.27)
-				)
-			)
-		)
-		(property "Footprint" ""
-			(at 251.46 97.79 0)
-			(effects
-				(font
-					(size 1.27 1.27)
-				)
-				(hide yes)
-			)
-		)
-		(property "Datasheet" ""
-			(at 251.46 97.79 0)
-			(effects
-				(font
-					(size 1.27 1.27)
-				)
-				(hide yes)
-			)
-		)
-		(property "Description" "Power symbol creates a global label with name \"+3.3V\""
-			(at 251.46 97.79 0)
-			(effects
-				(font
-					(size 1.27 1.27)
-				)
-				(hide yes)
-			)
-		)
-		(pin "1"
-		)
-		(instances
-			(project "pico-radio-5"
-				(path "/b9640508-dcc6-4f6b-830f-c53a732dcb5b"
-					(reference "#PWR011")
-					(unit 1)
-				)
-			)
-		)
-	)
-	(symbol
 		(lib_id "power:GND")
 		(at 22.86 73.66 0)
@@
 	)
 	(symbol
+		(lib_id "Jumper:SolderJumper_2_Open")
+		(at 128.27 64.77 0)
+		(unit 1)
+		(exclude_from_sim no)
+		(in_bom no)
+		(on_board yes)
+		(dnp no)
+		(fields_autoplaced yes)
+		(property "Reference" "JP3"
+			(at 128.27 58.42 0)
+			(effects
+				(font
+					(size 1.27 1.27)
+				)
+			)
+		)
+		(property "Value" "TFT SDO - ha kell"
+			(at 128.27 60.96 0)
+			(effects
+				(font
+					(size 1.27 1.27)
+				)
+			)
+		)
+		(property "Footprint" "Jumper:SolderJumper-2_P1.3mm_Open_RoundedPad1.0x1.5mm"
+			(at 128.27 64.77 0)
+			(effects
+				(font
+					(size 1.27 1.27)
+				)
+				(hide yes)
+			)
+		)
+		(property "Datasheet" "~"
+			(at 128.27 64.77 0)
+			(effects
+				(font
+					(size 1.27 1.27)
+				)
+				(hide yes)
+			)
+		)
+		(property "Description" "Solder Jumper, 2-pole, open"
+			(at 128.27 64.77 0)
+			(effects
+				(font
+					(size 1.27 1.27)
+				)
+				(hide yes)
+			)
+		)
+		(pin "1"
+		)
+		(pin "2"
+		)
+		(instances
+			(project ""
+				(path "/b9640508-dcc6-4f6b-830f-c53a732dcb5b"
+					(reference "JP3")
+					(unit 1)
+				)
+			)
+		)
+	)
+	(symbol
 		(lib_id "Device:Buzzer")
 		(at 254 102.87 0)
@@
 			)
 		)
-		(property "Value" "47uH"
+		(property "Value" "220uH"
 			(at 181.102 114.046 90)
 			(effects
@@
 			)
 		)
-		(property "Value" "200k"
+		(property "Value" "10k"
 			(at 240.03 69.8499 0)
 			(effects
@@
 			)
 		)
-		(property "Value" "100k"
+		(property "Value" "15k"
 			(at 240.03 81.2799 0)
 			(effects
@@
 			)
 		)
-		(property "Value" "270uH"
+		(property "Value" "220uH"
 			(at 55.626 76.454 0)
 			(effects
@@
 					(unit 1)
 				)
+			)
+		)
+	)
+	(symbol
+		(lib_id "power:+BATT")
+		(at 251.46 92.71 0)
+		(unit 1)
+		(exclude_from_sim no)
+		(in_bom yes)
+		(on_board yes)
+		(dnp no)
+		(property "Reference" "#PWR011"
+			(at 251.46 96.52 0)
+			(effects
+				(font
+					(size 1.27 1.27)
+				)
+				(hide yes)
+			)
+		)
+		(property "Value" "+Vbus"
+			(at 251.46 88.646 0)
+			(effects
+				(font
+					(size 1.27 1.27)
+				)
+			)
+		)
+		(property "Footprint" ""
+			(at 251.46 92.71 0)
+			(effects
+				(font
+					(size 1.27 1.27)
+				)
+				(hide yes)
+			)
+		)
+		(property "Datasheet" ""
+			(at 251.46 92.71 0)
+			(effects
+				(font
+					(size 1.27 1.27)
+				)
+				(hide yes)
+			)
+		)
+		(property "Description" "Power symbol creates a global label with name \"+BATT\""
+			(at 251.46 92.71 0)
+			(effects
+				(font
+					(size 1.27 1.27)
+				)
+				(hide yes)
+			)
+		)
+		(pin "1"
+		)
+		(instances
+			(project "pico-radio-5"
+				(path "/b9640508-dcc6-4f6b-830f-c53a732dcb5b"
+					(reference "#PWR011")
+					(unit 1)
+				)
